Commit message: - Made Changes in URDF

File: my_robot_description/urdf/my_robot.urdf (robot description, URDF)
Before this commit: robot my_robot, 5 links, 4 joints
Links:
- link base_link: geometry visual box size=${base_length} ${base_width} ${base_height}
- link caster_wheel: geometry visual sphere radius=${2*wheel_radius}
- link left_wheel_link: geometry visual cylinder length=${wheel_length} radius=${wheel_radius}
- link right_wheel_link: geometry visual cylinder length=${wheel_length} radius=${wheel_radius}
Joints:
- joint base_link_base_footprint_joint: origin xyz=0 0 0.1 rpy=0 0 0 -> xyz=0 0 ${wheel_length} rpy=0 0 0
- joint caster_wheel_base_joint: origin xyz=0.2 0 -0.15 rpy=0 0 0 -> xyz=${base_length/3.0} 0 -0.15 rpy=0 0 0
- joint left_wheel_base_joint: limit lower=-1.57 upper=1.57 effort=100 velocity=100 -> lower=-${pi/2.0} upper=${pi/2.0} effort=100 velocity=100; origin xyz=-0.15 0.225 -0.1 rpy=1.57 0 0 -> xyz=${-base_length / 4.0} ${(base_width + 0.05) / 2.0} -0.1 rpy=${pi / 2.0} 0 0
- joint right_wheel_base_joint: origin xyz=-0.15 -0.225 -0.1 rpy=1.57 0 0 -> xyz=${-base_length / 4.0} ${-(base_width + 0.05) / 2.0} -0.1 rpy=${pi/2.0}  0 0

Commit message: Added Xacro Macros for wheel_link

File: my_robot_description/urdf/my_robot.urdf (robot description, URDF)
Before this commit: robot my_robot, 5 links, 4 joints
Links:
- removed link left_wheel_link
- removed link right_wheel_link
- link caster_wheel: geometry visual sphere radius=${wheel_radius/2.0}
Joints:
- joint base_link_base_footprint_joint: origin xyz=0 0 ${wheel_length} rpy=0 0 0 -> xyz=0 0 -${wheel_length} rpy=0 0 0
- joint caster_wheel_base_joint: origin xyz=${base_length/3.0} 0 -0.15 rpy=0 0 0 -> xyz=${base_length/3.0} 0 -0.05 rpy=0 0 0
- joint left_wheel_base_joint: origin xyz=${-base_length / 4.0} ${(base_width + 0.05) / 2.0} -0.1 rpy=${pi / 2.0} 0 0 -> xyz=${-base_length / 4.0} ${(base_width + 0.05) / 2.0} 0 rpy=${pi / 2.0} 0 0
- joint right_wheel_base_joint: origin xyz=${-base_length / 4.0} ${-(base_width + 0.05) / 2.0} -0.1 rpy=${pi/2.0}  0 0 -> xyz=${-base_length / 4.0} ${-(base_width + 0.05) / 2.0} 0 rpy=${pi/2.0}  0 0

Commit message: Completed Xacro Structures

File: my_robot_description/urdf/my_robot.urdf (robot description, URDF)
Before this commit: robot my_robot, 3 links, 4 joints
Links:
- removed link base_footprint
- removed link base_link
- removed link caster_wheel
Joints:
- removed joint base_link_base_footprint_joint
- removed joint caster_wheel_base_joint
- removed joint left_wheel_base_joint
- removed joint right_wheel_base_joint
