Commit message: Fixed  Collision changes in urdf files

File: my_robot_description/urdf/mobile_base.xacro (robot description, xacro)
@@ -15,4 +15,12 @@
             <material name="blue" />
         </visual>
+        <collision>
+                <geometry>
+                    <geometry>
+                        <box size="${base_length} ${base_width} ${base_height}"/>
+                    </geometry>
+                </geometry>
+                <origin xyz="0.0 0.0 0.0" rpy="0.0 0.0 0.0"/>
+        </collision>
         <xacro:box_inertia m="5.0" l="${2*base_length}" w="${2*base_width}" h="${2*base_height}"
                            xyz="0 0 ${base_height / 2.0}" rpy="0 0 0" />
@@ -27,4 +35,10 @@
                 <material name="grey" />
             </visual>
+            <collision>
+                <geometry>
+                    <cylinder radius ="${wheel_radius}" length="${wheel_length}"/>
+                </geometry>
+                <origin xyz="0.0 0.0 0.0" rpy="0.0 0.0 0.0"/>
+            </collision>
             <xacro:cylinder_inertia m="1.0" r="${2*wheel_radius}" h="${2*wheel_length}" xyz="0 0 0" rpy="${pi/2.0} 0 0" />
         </link>
@@ -41,8 +55,8 @@
         </visual>
         <collision>
-                <geometry>
-                    <sphere radius="${wheel_radius/2.0}"/>
-                </geometry>
-                <origin xyz="0.0 0.0 0.0" rpy="0.0 0.0 0.0"/>
+            <geometry>
+                <sphere radius="${wheel_radius/2.0}"/>
+            </geometry>
+            <origin xyz="0.0 0.0 0.0" rpy="0.0 0.0 0.0"/>
         </collision>
         <xacro:sphere_inertia m="0.5" r="${2*wheel_radius / 2.0}"

File: my_robot_description/urdf/mobile_base_gazebo.xacro (robot description, xacro)
@@ -4,3 +4,12 @@
         <material>Gazebo/Blue</material>
     </gazebo>
+    <gazebo reference="right_wheel_link">
+        <material>Gazebo/Grey</material>
+    </gazebo>
+    <gazebo reference="left_wheel_link">
+        <material>Gazebo/Grey</material>
+    </gazebo>
+    <gazebo reference="caster_wheel_link">
+        <material>Gazebo/Grey</material>
+    </gazebo>
 </robot>

Commit message: Added Following Things -  Added Diff Drive Control Plugin - Added Coeeficient of Friction tags to reduce Caster wheel friction

File: my_robot_description/urdf/mobile_base.xacro (robot description, xacro)
@@ -21,5 +21,5 @@
                     </geometry>
                 </geometry>
-                <origin xyz="0.0 0.0 0.0" rpy="0.0 0.0 0.0"/>
+                <origin xyz="0 0 ${base_height / 2.0}" rpy="0 0 0"/>
         </collision>
         <xacro:box_inertia m="5.0" l="${2*base_length}" w="${2*base_width}" h="${2*base_height}"
@@ -39,5 +39,5 @@
                     <cylinder radius ="${wheel_radius}" length="${wheel_length}"/>
                 </geometry>
-                <origin xyz="0.0 0.0 0.0" rpy="0.0 0.0 0.0"/>
+                <origin xyz="0 0 0" rpy="${pi / 2.0} 0 0"/>
             </collision>
             <xacro:cylinder_inertia m="1.0" r="${2*wheel_radius}" h="${2*wheel_length}" xyz="0 0 0" rpy="${pi/2.0} 0 0" />
@@ -58,5 +58,5 @@
                 <sphere radius="${wheel_radius/2.0}"/>
             </geometry>
-            <origin xyz="0.0 0.0 0.0" rpy="0.0 0.0 0.0"/>
+            <origin xyz="0 0 0" rpy="0 0 0"/>
         </collision>
         <xacro:sphere_inertia m="0.5" r="${2*wheel_radius / 2.0}"

File: my_robot_description/urdf/mobile_base_gazebo.xacro (robot description, xacro)
@@ -12,4 +12,27 @@
     <gazebo reference="caster_wheel_link">
         <material>Gazebo/Grey</material>
+        <mu1 value="0.1"/>
+        <mu2 value="0.1"/>
+    </gazebo>
+    <gazebo>
+        <plugin name="gazebo_ros_diff_drive" filename="libgazebo_ros_diff_drive.so">
+        <!-- Update rate in Hz -->
+        <update_rate>50</update_rate>
+        <!-- wheels -->
+        <left_joint>base_left_wheel_joint</left_joint>
+        <right_joint>base_right_wheel_joint</right_joint>
+        <!-- kinematics -->
+        <wheel_separation>0.45</wheel_separation>
+        <wheel_diameter>0.2</wheel_diameter>
+        <!-- input -->
+        <command_topic>cmd_vel</command_topic>
+        <!-- output -->
+        <publish_odom>true</publish_odom>
+        <publish_odom_tf>true</publish_odom_tf>
+        <publish_wheel_tf>true</publish_wheel_tf>
+        <odometry_topic>odom</odometry_topic>
+        <odometry_frame>odom</odometry_frame>
+        <robot_base_frame>base_footprint</robot_base_frame>
+        </plugin>
     </gazebo>
 </robot>

Commit message: Added Following things - Added Camera Links - Added Camera Plugin - Added My World

File: my_robot_description/urdf/mobile_base.xacro (robot description, xacro)
@@ -16,10 +16,8 @@
         </visual>
         <collision>
-                <geometry>
-                    <geometry>
-                        <box size="${base_length} ${base_width} ${base_height}"/>
-                    </geometry>
-                </geometry>
-                <origin xyz="0 0 ${base_height / 2.0}" rpy="0 0 0"/>
+            <geometry>
+                <box size="${base_length} ${base_width} ${base_height}" />
+            </geometry>
+            <origin xyz="0 0 ${base_height / 2.0}" rpy="0 0 0" />
         </collision>
         <xacro:box_inertia m="5.0" l="${2*base_length}" w="${2*base_width}" h="${2*base_height}"
@@ -37,9 +35,10 @@
             <collision>
                 <geometry>
-                    <cylinder radius ="${wheel_radius}" length="${wheel_length}"/>
+                    <cylinder radius="${wheel_radius}" length="${wheel_length}" />
                 </geometry>
-                <origin xyz="0 0 0" rpy="${pi / 2.0} 0 0"/>
+                <origin xyz="0 0 0" rpy="${pi / 2.0} 0 0" />
             </collision>
-            <xacro:cylinder_inertia m="1.0" r="${2*wheel_radius}" h="${2*wheel_length}" xyz="0 0 0" rpy="${pi/2.0} 0 0" />
+            <xacro:cylinder_inertia m="1.0" r="${2*wheel_radius}" h="${2*wheel_length}"
+                                    xyz="0 0 0" rpy="${pi / 2.0} 0 0" />
         </link>
     </xacro:macro>
@@ -56,7 +55,7 @@
         <collision>
             <geometry>
-                <sphere radius="${wheel_radius/2.0}"/>
+                <sphere radius="${wheel_radius / 2.0}" />
             </geometry>
-            <origin xyz="0 0 0" rpy="0 0 0"/>
+            <origin xyz="0 0 0" rpy="0 0 0" />
         </collision>
         <xacro:sphere_inertia m="0.5" r="${2*wheel_radius / 2.0}"

File: my_robot_description/urdf/mobile_base_gazebo.xacro (robot description, xacro)
@@ -12,26 +12,24 @@
     <gazebo reference="caster_wheel_link">
         <material>Gazebo/Grey</material>
-        <mu1 value="0.1"/>
-        <mu2 value="0.1"/>
+        <mu1 value="0.1" />
+        <mu2 value="0.1" />
     </gazebo>
     <gazebo>
-        <plugin name="gazebo_ros_diff_drive" filename="libgazebo_ros_diff_drive.so">
-        <!-- Update rate in Hz -->
-        <update_rate>50</update_rate>
-        <!-- wheels -->
-        <left_joint>base_left_wheel_joint</left_joint>
-        <right_joint>base_right_wheel_joint</right_joint>
-        <!-- kinematics -->
-        <wheel_separation>0.45</wheel_separation>
-        <wheel_diameter>0.2</wheel_diameter>
-        <!-- input -->
-        <command_topic>cmd_vel</command_topic>
-        <!-- output -->
-        <publish_odom>true</publish_odom>
-        <publish_odom_tf>true</publish_odom_tf>
-        <publish_wheel_tf>true</publish_wheel_tf>
-        <odometry_topic>odom</odometry_topic>
-        <odometry_frame>odom</odometry_frame>
-        <robot_base_frame>base_footprint</robot_base_frame>
+        <plugin name="diff_drive_controller" filename="libgazebo_ros_diff_drive.so">
+            <!-- Update rate in Hz -->
+            <update_rate>50</update_rate>
+            <!-- wheels -->
+            <left_joint>base_left_wheel_joint</left_joint>
+            <right_joint>base_right_wheel_joint</right_joint>
+            <!-- kinematics -->
+            <wheel_separation>0.45</wheel_separation>
+            <wheel_diameter>0.2</wheel_diameter>
+            <!-- output -->
+            <publish_odom>true</publish_odom>
+            <publish_odom_tf>true</publish_odom_tf>
+            <publish_wheel_tf>true</publish_wheel_tf>
+            <odometry_topic>odom</odometry_topic>
+            <odometry_frame>odom</odometry_frame>
+            <robot_base_frame>base_footprint</robot_base_frame>
         </plugin>
     </gazebo>
