Commit message: Made following changes - Added Joint State Publisher Plugin - Added Joint State Trajectory Plugin - Visualized TFs

File: my_robot_description/urdf/arm.xacro (robot description, xacro)
@@ -1,60 +1,77 @@
 <?xml version="1.0"?>
 <robot xmlns:xacro="http://www.ros.org/wiki/xacro">
-    <!-- Xacros-->
-    <xacro:property name="arm_base_side" value="0.1"/>
-    <xacro:property name="arm_base_height" value="0.02"/>
-    <xacro:property name="arm_length" value="0.3"/>
-    <xacro:property name="arm_radius" value="0.02"/>
-    <!-- Links-->
+    <xacro:property name="arm_base_length" value="0.1" />
+    <xacro:property name="arm_base_width" value="0.1" />
+    <xacro:property name="arm_base_height" value="0.02" />
+    <xacro:property name="forearm_radius" value="0.02" />
+    <xacro:property name="forearm_length" value="0.3" />
+    <xacro:property name="hand_radius" value="0.02" />
+    <xacro:property name="hand_length" value="0.3" />
     <link name="arm_base_link">
-        <geometry>
-            <box size="${arm_base_side} ${arm_base_side} ${arm_base_height}"/>
-            <origin xyz="0 0 0" rpy="0 0 0"/>
-        </geometry>
+        <visual>
+            <geometry>
+                <box size="${arm_base_length} ${arm_base_width} ${arm_base_height}" />
+            </geometry>
+            <origin xyz="0 0 ${arm_base_height / 2.0}" rpy="0 0 0" />
+            <material name="orange" />
+        </visual>
         <collision>
-            <box size="${arm_base_side} ${arm_base_side} ${arm_base_height}"/>
-            <origin xyz="0 0 0" rpy="0 0 0"/>
+            <geometry>
+                <box size="${arm_base_length} ${arm_base_width} ${arm_base_height}" />
+            </geometry>
+            <origin xyz="0 0 ${arm_base_height / 2.0}" rpy="0 0 0" />
         </collision>
-        <xacro:box_intertia m="0.5" l="${arm_base_side}" w="${arm_base_side}" h="${arm_base_height}"
-                             xyz="0 0 0" rpy="0 0 0" />
+        <xacro:box_inertia m="0.5" l="${2*arm_base_length}" w="${2*arm_base_width}" h="${2*arm_base_height}"
+                           xyz="0 0 ${arm_base_height / 2.0}" rpy="0 0 0" />
     </link>
     <link name="forearm_link">
-        <geometry>
-            <cylinder radius="${arm_radius}" length="${arm_length}"/>
-            <origin xyz="0 0 0" rpy="0 0 0"/>
-        </geometry>
+        <visual>
+            <geometry>
+                <cylinder radius="${forearm_radius}" length="${forearm_length}" />
+            </geometry>
+            <origin xyz="0 0 ${forearm_length / 2.0}" rpy="0 0 0" />
+            <material name="yellow" />
+        </visual>
         <collision>
-            <origin xyz="0.0 0.0 0.0" rpy="0.0 0.0 0.0"/>
-            <cylinder radius="${arm_radius}" length="${arm_length}"/>
+            <geometry>
+                <cylinder radius="${forearm_radius}" length="${forearm_length}" />
+            </geometry>
+            <origin xyz="0 0 ${forearm_length / 2.0}" rpy="0 0 0" />
         </collision>
-        <xacro:cylinder_inertia m="0.3" r="${arm_radius}" h="${arm_length}" xyz="0 0 0" rpy="0 0 0"/>
+        <xacro:cylinder_inertia m="0.3" r="${2*forearm_radius}" h="${2*forearm_length}"
+                                xyz="0 0 ${forearm_length / 2.0}" rpy="0 0 0" />
     </link>
     <link name="hand_link">
-        <geometry>
-            <cylinder radius="${arm_radius}" length="${arm_length}"/>
-            <origin xyz="0 0 0" rpy="0 0 0"/>
-        </geometry>
+        <visual>
+            <geometry>
+                <cylinder radius="${hand_radius}" length="${hand_length}" />
+            </geometry>
+            <origin xyz="0 0 ${hand_length / 2.0}" rpy="0 0 0" />
+            <material name="orange" />
+        </visual>
         <collision>
-            <origin xyz="0.0 0.0 0.0" rpy="0.0 0.0 0.0"/>
-            <cylinder radius="${arm_radius}" length="${arm_length}"/>
+             <geometry>
+                <cylinder radius="${hand_radius}" length="${hand_length}" />
+            </geometry>
+            <origin xyz="0 0 ${hand_length / 2.0}" rpy="0 0 0" />
         </collision>
-        <xacro:cylinder_inertia m="0.3" r="${arm_radius}" h="${arm_length}" xyz="0 0 0" rpy="0 0 0"/>
+        <xacro:cylinder_inertia m="0.3" r="${2*hand_radius}" h="${2*hand_length}"
+                                xyz="0 0 ${hand_length / 2.0}" rpy="0 0 0" />
     </link>
-    <!-- Joints -->
     <joint name="arm_base_forearm_joint" type="revolute">
-        <origin xyz="0.0 0.0 0.0" rpy="0.0 0.0 0.0"/>
-        <parent link="arm_base_link"/>
-        <child link="forearm_link"/>
-        <axis xyz="0.0 0.0 0.0"/>
-        <limit lower="0.0" upper="${pi / 2.0}" effort="100" velocity="100"/>
-        <dynamics friction="0.05" damping="0.1"/>
+        <parent link="arm_base_link" />
+        <child link="forearm_link" />
+        <origin xyz="0 0 ${arm_base_height}" rpy="0 0 0" />
+        <axis xyz="0 1 0" />
+        <limit lower="0" upper="${pi/2}" effort="100" velocity="100" />
+        <dynamics friction="0.05" damping="0.1" />
     </joint>
     <joint name="forearm_hand_joint" type="revolute">
-        <origin xyz="0.0 0.0 0.0" rpy="0.0 0.0 0.0"/>
-        <parent link="forearm_link"/>
-        <child link="hand_link"/>
-        <axis xyz="0.0 0.0 0.0"/>
-        <limit lower="0.0" upper="${pi / 2.0}" effort="100" velocity="100"/>
-        <dynamics friction="0.05" damping="0.1"/>
+        <parent link="forearm_link" />
+        <child link="hand_link" />
+        <origin xyz="0 0 ${forearm_length}" rpy="0 0 0" />
+        <axis xyz="0 1 0" />
+        <limit lower="0" upper="${pi/2}" effort="100" velocity="100" />
+        <dynamics friction="0.05" damping="0.1" />
     </joint>
 </robot>

File: my_robot_description/urdf/standalone_arm.urdf.xacro (robot description, xacro)
@@ -1,5 +1,6 @@
 <?xml version="1.0"?>
-<robot name="arm" xmlns:xacro="https://www.ros.org/wiki/xacro">
+<robot name="my_robot" xmlns:xacro="http://www.ros.org/wiki/xacro">
     <xacro:include filename="common_properties.xacro" />
     <xacro:include filename="arm.xacro" />
+    <xacro:include filename="arm_gazebo.xacro" />
 </robot>
