Commit message: Differential Drive Final Commit

File: my_robot_description/urdf/my_robot.urdf.xacro (robot description, xacro)
@@ -5,3 +5,11 @@
     <xacro:include filename="mobile_base_gazebo.xacro" />
     <xacro:include filename="camera.xacro" />
+    <xacro:include filename="arm.xacro"/>
+    <xacro:include filename="arm_gazebo.xacro"/>
+    <joint name="base_arm_base_joint" type="fixed">
+        <parent link="base_link" />
+        <child link="arm_base_link" />
+        <origin xyz="${base_length / 4.0} 0 ${base_height}" rpy="0 0 0" />
+        <axis xyz="0 1 0" />
+    </joint>
 </robot>
